File: 8f2o/esp-switch.kicad_pcb (KiCad board)
At the start: 2 copper layers, 87.7 x 49.7 mm, 58 parts, among them J2 Screw_Terminal_01x04, J3 Screw_Terminal_01x04, J4 Conn_02x04_Odd_Even, J5 Screw_Terminal_01x04, J7 Screw_Terminal_01x04, Q1 TSM2302CX, Q2 TSM2302CX, Q3 TSM2302CX, Q4 TSM2302CX, Q5 TSM2302CX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

Commit message: v0.1 for 8f2o and 4f2t2o
Parts:
- removed J4: Conn_02x04_Odd_Even, Connector_PinHeader_2.54mm:PinHeader_2x04_P2.54mm_Vertical
- added J1: Conn_01x07_Socket, Connector_PinSocket_2.54mm:PinSocket_1x07_P2.54mm_Horizontal, F.Cu at (47.5, 39.4)
- added Q10: BC817, Package_TO_SOT_SMD:SOT-23_Handsoldering, F.Cu at (49.4, 33.3)
- added Q9: BC817, Package_TO_SOT_SMD:SOT-23_Handsoldering, B.Cu at (56.4, 43.7)
- added R25: 10k, Resistor_SMD:R_0805_2012Metric_Pad1.20x1.40mm_HandSolder, B.Cu at (53.1, 44.2)
- added R26: 10k, Resistor_SMD:R_0805_2012Metric_Pad1.20x1.40mm_HandSolder, F.Cu at (48.5, 36.4)
- C9: value 47n -> 100n; moved to B.Cu
- R10, R13, R14, R23, R9: moved to B.Cu
- moved R17 24.8 mm to (23.9, 42.4), turned to -90 degrees
- moved R22 24.7 mm to (23.9, 38.4), turned to 90 degrees
- moved R9 19.3 mm to (39.9, 27.5)
- moved R14 14.3 mm to (34.8, 27.5), turned to 90 degrees
- moved C5 13.4 mm to (42.7, 19.7)
- moved R15 12.7 mm to (40.5, 17.4), turned to 180 degrees
- moved R13 11.4 mm to (37.3, 27.5), turned to 90 degrees
- moved R23 10.8 mm to (50.0, 44.2), turned to -90 degrees
- moved C9 10.3 mm to (60.2, 43.2), turned to 90 degrees
- moved R10 6.75 mm to (62.7, 43.2)
- moved Q7 6.53 mm to (27.0, 22.4), turned to 180 degrees
- moved R16 6.11 mm to (40.5, 15.1), turned to 180 degrees
- moved Q6 3.88 mm to (27.0, 17.4), turned to 180 degrees
- moved C6 3.44 mm to (45.5, 25.5), turned to 90 degrees
- moved R24 3.36 mm to (45.2, 35.6), turned to 90 degrees
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Connections:
- C10 pad 1: /GPIO10 -> /GPIO12
- C11 pad 1: /GPIO9 -> /GPIO13
- Q1 pad 1: /GPIO14 -> /GPIO10
- Q2 pad 1: /GPIO13 -> /GPIO14
- Q3 pad 1: /GPIO12 -> /GPIO9
- R15 pad 2: /GPIO10 -> /GPIO12
- R16 pad 2: /GPIO9 -> /GPIO13
- R23 pad 1: /GPIO2 -> Net-(J1-Pin_2)
- R24 pad 1: /GPIO0 -> Net-(J1-Pin_1)
- R3 pad 2: /GPIO14 -> /GPIO10
- R4 pad 2: /GPIO13 -> /GPIO14
- R5 pad 2: /GPIO12 -> /GPIO9
- U3 pad 4: /GPIO10 -> /GPIO12
- U4 pad 4: /GPIO9 -> /GPIO13
Routing:
- net GND: track 34.5 -> 4.99 mm, vias 61 -> 60
- net /GPIO13: track 47.2 -> 21.8 mm, vias 1 -> 0
- net Net-(J1-Pin_3): track 6.94 -> 30.4 mm
- net +3V3: track 57.6 -> 39.7 mm, vias 0 -> 1
- net /GPIO2: track 40.4 -> 24.3 mm, vias 1 -> 2
- net /GPIO3: track 18.8 -> 3.40 mm
- net Net-(J1-Pin_4): track 19.7 -> 34.9 mm
- net /GPIO1: track 18.9 -> 4.99 mm
- net /GPIO14: track 60.2 -> 46.6 mm
- net /GPIO12: track 46.9 -> 33.4 mm, vias 1 -> 0
- net /GPIO10: track 31.4 -> 42.6 mm, vias 0 -> 1
- net /GPIO9: track 21.9 -> 33.0 mm, vias 2 -> 1
- net /EN: track 19.7 -> 10.3 mm, vias 2 -> 1
- net /nRST: track 24.4 -> 30.9 mm
- net Net-(Q10-E): track 21.1 -> 14.9 mm
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Other:
- board text added: "JLCJLCJLCJLC"
- board text added: "esp-switch-8f2o v0.2"
- board text removed: "GND"
