File: 8f2o/esp-switch.kicad_sch (KiCad schematic)
At the start: 58 parts, among them J2 Screw_Terminal_01x04, J3 Screw_Terminal_01x04, J4 Conn_02x04_Odd_Even, J5 Screw_Terminal_01x04, J7 Screw_Terminal_01x04, Q1 TSM2302CX, Q2 TSM2302CX, Q3 TSM2302CX, Q4 TSM2302CX, Q5 TSM2302CX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

Commit message: v0.1 for 8f2o and 4f2t2o
Parts:
- removed J4: Conn_02x04_Odd_Even, Connector_PinHeader_2.54mm:PinHeader_2x04_P2.54mm_Vertical, symbol Connector_Generic:Conn_02x04_Odd_Even
- added J1: Conn_01x07_Socket, Connector_PinSocket_2.54mm:PinSocket_1x07_P2.54mm_Horizontal, symbol Connector:Conn_01x07_Socket
- added Q10, Q9: BC817, Package_TO_SOT_SMD:SOT-23_Handsoldering, symbol Simulation_SPICE:NPN
- added R25, R26: 10k, Resistor_SMD:R_0805_2012Metric_Pad1.20x1.40mm_HandSolder, symbol Device:R
- C9: value 47n -> 100n
Connections:
- net +3V3: now also J1.7 (Pin_7)
- net GND: now also J1.6 (Pin_6)
- net GPIO0: now also Q10.1 (C); no longer R24.1
- net GPIO10: now also Q1.1 (G), R3.2; no longer C10.1, R15.2, U3.4
- net GPIO12: now also C10.1, R15.2, U3.4; no longer Q3.1 (G), R5.2
- net GPIO13: now also C11.1, R16.2, U4.4; no longer Q2.1 (G), R4.2
- net GPIO14: now also Q2.1 (G), R4.2; no longer Q1.1 (G), R3.2
- net GPIO2: no longer R23.1
- net GPIO9: now also Q3.1 (G), R5.2; no longer C11.1, R16.2, U4.4
- net nRST: now also Q9.1 (C)
- net at R23.2: now also Q10.3 (E), R25.1
- net at R17.1: now also J1.3 (Pin_3)
- net at R24.2: now also Q9.3 (E), R26.1
- net at R22.2: now also J1.4 (Pin_4)
- new net: Q9.2 (B), R25.2
- new net: J1.1 (Pin_1), R24.1
- new net: J1.2 (Pin_2), R23.1
- new net: Q10.2 (B), R26.2
- no-connect marks 6 -> 7
Other:
- moved on the sheet: C10, C11, C5, D1, D2, J7, R15, R16, R17, R18, R19, R20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

Commit message: Updates
Other:
- note added: "HIGH AT BOOT"
- note added: "Incorrect footprint"
- note added: "MOVE TO GPIO16"
Changed lines of the file:
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@@
     (stroke (width 0) (type default))
+  )
+  (text "Incorrect footprint" (at 210.185 120.015 0)
+    (effects (font (size 1.27 1.27)) (justify left bottom))
+  )
+  (text "HIGH AT BOOT" (at 117.475 141.605 0)
+    (effects (font (size 1.27 1.27)) (justify left bottom))
+  )
+  (text "Incorrect footprint" (at 212.09 137.795 0)
+    (effects (font (size 1.27 1.27)) (justify left bottom))
+  )
+  (text "MOVE TO GPIO16" (at 29.845 161.29 0)
+    (effects (font (size 1.27 1.27)) (justify left bottom))
+  )
+  (text "HIGH AT BOOT" (at 118.11 162.56 0)
+    (effects (font (size 1.27 1.27)) (justify left bottom))
+  )
+  (text "HIGH AT BOOT" (at 27.305 164.465 0)
+    (effects (font (size 1.27 1.27)) (justify left bottom))
   )
   (label "GPIO3" (at 170.18 46.99 180) (fields_autoplaced)
