File: 4f2t2o/esp-switch.kicad_pcb (KiCad board)
At the start: 2 copper layers, 87.7 x 49.7 mm, 62 parts, among them J2 Screw_Terminal_01x04, J3 Screw_Terminal_01x04, J4 Conn_02x04_Odd_Even, J5 Screw_Terminal_01x04, J7 Screw_Terminal_01x04, Q1 TSM2302CX, Q2 TSM2302CX, Q3 TSM2302CX, Q4 TSM2302CX, Q5 BT138-600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

Commit message: v0.1 for 8f2o and 4f2t2o
Parts:
- removed J4: Conn_02x04_Odd_Even, Connector_PinHeader_2.54mm:PinHeader_2x04_P2.54mm_Vertical
- removed R17, R22, R23, R24: 10R, Resistor_SMD:R_0805_2012Metric_Pad1.20x1.40mm_HandSolder
- removed RV1, RV2: Varistor, Varistor:RV_Disc_D7mm_W5.7mm_P5mm
- added D4: SMAJ400CA, Diode_SMD:D_SMA, F.Cu at (74.2, 3.77)
- added D5: SMAJ400CA, Diode_SMD:D_SMA, F.Cu at (74.2, 11.3)
- added D6: SMAJ400CA, Diode_SMD:D_SMA, F.Cu at (13.5, 3.76)
- added D7: SMAJ400CA, Diode_SMD:D_SMA, F.Cu at (13.5, 11.3)
- added J1: Conn_01x07_Socket, Connector_PinSocket_2.54mm:PinSocket_1x07_P2.54mm_Horizontal, F.Cu at (47.5, 39.4)
- added Q7: BC817, Package_TO_SOT_SMD:SOT-23_Handsoldering, B.Cu at (56.4, 43.7)
- added Q8: BC817, Package_TO_SOT_SMD:SOT-23_Handsoldering, F.Cu at (49.5, 33.1)
- added R29: 10k, Resistor_SMD:R_0805_2012Metric_Pad1.20x1.40mm_HandSolder, B.Cu at (53.1, 44.2)
- added R30: 10k, Resistor_SMD:R_0805_2012Metric_Pad1.20x1.40mm_HandSolder, F.Cu at (49.0, 36.2)
- added R31: 10R, Resistor_SMD:R_0805_2012Metric_Pad1.20x1.40mm_HandSolder, F.Cu at (23.9, 42.4)
- added R32: 220, Resistor_SMD:R_0805_2012Metric_Pad1.20x1.40mm_HandSolder, B.Cu at (50.0, 44.2)
- added R33: 220, Resistor_SMD:R_0805_2012Metric_Pad1.20x1.40mm_HandSolder, F.Cu at (45.0, 35.6)
- added R34: 10R, Resistor_SMD:R_0805_2012Metric_Pad1.20x1.40mm_HandSolder, F.Cu at (23.9, 38.4)
- C5, C9, R10, R13, R14, R15, R16: moved to B.Cu
- Q5, Q6: footprint Package_TO_SOT_THT:TO-220-3_Vertical -> esp-switch:TO-220-3_Vertical_offset
- R11, R26: value 200 -> 220
- moved R15 23.1 mm to (39.6, 27.6), turned to -90 degrees
- moved R4 20.4 mm to (33.0, 37.8)
- moved R3 19.2 mm to (30.5, 37.8), turned to 90 degrees
- moved C5 19.1 mm to (42.3, 26.4), turned to 90 degrees
- moved R16 16.7 mm to (37.3, 27.6), turned to -90 degrees
- moved R14 16.2 mm to (32.8, 27.6), turned to 90 degrees
- moved R5 15.9 mm to (35.4, 37.8)
- moved R13 13.6 mm to (35.1, 27.6), turned to 90 degrees
- moved R9 12.8 mm to (45.0, 31.6)
- moved C9 10.3 mm to (60.2, 43.2), turned to 90 degrees
- moved R10 6.75 mm to (62.7, 43.2)
- moved R11 6.15 mm to (41.6, 17.1)
- moved U1 6.14 mm to (40.2, 3.73)
- moved U6 6.14 mm to (40.2, 11.3)
- moved R26 6.14 mm to (44.0, 17.1)
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Connections:
- C10 pad 1: /GPIO10 -> /GPIO13
- C11 pad 1: /GPIO9 -> /GPIO12
- J2 pad 1: Net-(J2-Pin_1) -> Net-(D6-A2)
- J2 pad 4: Net-(J2-Pin_4) -> Net-(D7-A2)
- Q5 pad 1: Net-(J2-Pin_1) -> Net-(D6-A2)
- Q6 pad 1: Net-(J2-Pin_4) -> Net-(D7-A2)
- R11 pad 1: /GPIO12 -> /GPIO10
- R12 pad 1: Net-(R12-Pad1) -> Net-(Q5-G)
- R12 pad 2: Net-(Q5-G) -> Net-(D6-A2)
- R15 pad 2: /GPIO10 -> /GPIO13
- R16 pad 2: /GPIO9 -> /GPIO12
- R26 pad 1: /GPIO13 -> /GPIO9
- R27 pad 1: Net-(R27-Pad1) -> Net-(Q6-G)
- R27 pad 2: Net-(Q6-G) -> Net-(D7-A2)
- U1 pad 4: Net-(R12-Pad1) -> Net-(Q5-G)
- U3 pad 4: /GPIO10 -> /GPIO13
- U4 pad 4: /GPIO9 -> /GPIO12
- U6 pad 4: Net-(R27-Pad1) -> Net-(Q6-G)
Routing:
- net Net-(J1-Pin_4): track 0.00 -> 35.4 mm
- net Net-(J1-Pin_3): track 0.00 -> 31.1 mm
- net Net-(D6-A2): track 0.00 -> 30.3 mm
- net Net-(D7-A2): track 0.00 -> 25.4 mm
- net /GPIO10: track 34.2 -> 11.8 mm, vias 1 -> 0
- net Net-(J4-Pin_4): track 19.6 -> 0.00 mm, vias 1 -> 0
- net Net-(J4-Pin_6): track 19.1 -> 0.00 mm, vias 1 -> 0
- net Net-(J4-Pin_2): track 17.6 -> 0.00 mm
- net Net-(Q7-E): track 0.00 -> 17.4 mm, vias 0 -> 1
- net /GPIO3: track 18.8 -> 3.40 mm
- net Net-(Q8-E): track 0.00 -> 15.1 mm, vias 0 -> 1
- net /GPIO13: track 19.4 -> 33.9 mm, vias 0 -> 1
- net /GPIO9: track 26.4 -> 12.8 mm, vias 1 -> 0
- net /GPIO2: track 21.0 -> 7.61 mm, vias 0 -> 1
- net /GPIO1: track 18.9 -> 5.53 mm
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Other:
- board text added: "JLCJLCJLCJLC"
- board text added: "esp-switch-4f2t2o v0.1"
- board text removed: "GND"

Commit message: Updates
Parts:
- Q5, Q6: footprint esp-switch:TO-220-3_Vertical_offset -> Package_TO_SOT_SMD:TO-252-2
- R1: value 68k -> 150k
- R10, R13, R14, R2, R29, R3, R30, R4, R5, R6, R9: value 10k -> 22k
- R32, R33: value 220 -> 10R
- moved R11 20.1 mm to (47.4, -2.13), turned to 180 degrees
- moved R26 9.08 mm to (47.2, 8.62)
- moved Q5 3.55 mm to (22.9, 3.81)
- moved Q6 3.51 mm to (22.9, 11.4)
- moved R12 2.09 mm to (29.8, 5.59), turned to 0 degrees
- moved R27 2.09 mm to (29.8, 13.2), turned to 0 degrees
- moved C11 1.40 mm to (47.2, 12.7)
Connections:
- Q1 pad 1: /GPIO5 -> /GPIO2
- Q2 pad 1: /GPIO4 -> /GPIO0
- Q5 pad 1: Net-(D6-A2) -> Net-(D6-A1)
- Q5 pad 2: Net-(D6-A1) -> Net-(D6-A2)
- Q6 pad 1: Net-(D7-A2) -> Net-(D7-A1)
- Q6 pad 2: Net-(D7-A1) -> Net-(D7-A2)
- R11 pad 1: /GPIO10 -> GND
- R11 pad 2: Net-(U1-A) -> Net-(U1-K)
- R12 pad 2: Net-(D6-A2) -> Net-(D6-A1)
- R25 pad 1: Net-(D6-A1) -> Net-(D6-A2)
- R26 pad 1: /GPIO9 -> GND
- R26 pad 2: Net-(U6-A) -> Net-(U6-K)
- R27 pad 2: Net-(D7-A2) -> Net-(D7-A1)
- R28 pad 1: Net-(D7-A1) -> Net-(D7-A2)
- R3 pad 2: /GPIO5 -> /GPIO2
- R4 pad 2: /GPIO4 -> /GPIO0
- U1 pad 1: Net-(U1-A) -> /GPIO5
- U1 pad 2: GND -> Net-(U1-K)
- U6 pad 1: Net-(U6-A) -> /GPIO4
- U6 pad 2: GND -> Net-(U6-K)
Routing:
- net /GPIO2: track 7.61 -> 24.8 mm
- net /GPIO0: track 24.8 -> 41.4 mm
- net /GPIO9: track 12.8 -> 0.00 mm
- net Net-(U1-A): track 12.1 -> 0.00 mm
- net /GPIO10: track 11.8 -> 0.00 mm
- net Net-(Q5-G): track 13.4 -> 24.1 mm, vias 0 -> 1
- net Net-(Q6-G): track 13.7 -> 24.1 mm, vias 0 -> 1
- net Net-(D6-A2): track 30.3 -> 24.0 mm
- net Net-(U6-A): track 3.54 -> 0.00 mm
- net Net-(D7-A1): track 25.8 -> 29.1 mm, vias 0 -> 1
- net Net-(D6-A1): track 25.3 -> 28.2 mm, vias 0 -> 1
- net Net-(D7-A2): track 25.4 -> 22.8 mm
- net /GPIO12: track 30.2 -> 27.6 mm
- net GND: vias 49 -> 45
Other:
- board text added: "esp-switch-4f2t2o v0.2"
