File: 4f2t2o/esp-switch.kicad_sch (KiCad schematic)
At the start: 62 parts, among them J2 Screw_Terminal_01x04, J3 Screw_Terminal_01x04, J4 Conn_02x04_Odd_Even, J5 Screw_Terminal_01x04, J7 Screw_Terminal_01x04, Q1 TSM2302CX, Q2 TSM2302CX, Q3 TSM2302CX, Q4 TSM2302CX, Q5 BT138-600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

Commit message: v0.1 for 8f2o and 4f2t2o
Parts:
- removed J4: Conn_02x04_Odd_Even, Connector_PinHeader_2.54mm:PinHeader_2x04_P2.54mm_Vertical, symbol Connector_Generic:Conn_02x04_Odd_Even
- removed R17, R22, R23, R24: 10R, Resistor_SMD:R_0805_2012Metric_Pad1.20x1.40mm_HandSolder, symbol Device:R
- removed RV1, RV2: Varistor, Varistor:RV_Disc_D7mm_W5.7mm_P5mm, symbol Device:Varistor
- added D4, D5, D6, D7: SMAJ400CA, Diode_SMD:D_SMA, symbol Diode:SMAJ400CA
- added J1: Conn_01x07_Socket, Connector_PinSocket_2.54mm:PinSocket_1x07_P2.54mm_Horizontal, symbol Connector:Conn_01x07_Socket
- added Q7, Q8: BC817, Package_TO_SOT_SMD:SOT-23_Handsoldering, symbol Simulation_SPICE:NPN
- added R29, R30: 10k, Resistor_SMD:R_0805_2012Metric_Pad1.20x1.40mm_HandSolder, symbol Device:R
- added R31, R34: 10R, Resistor_SMD:R_0805_2012Metric_Pad1.20x1.40mm_HandSolder, symbol Device:R
- added R32, R33: 220, Resistor_SMD:R_0805_2012Metric_Pad1.20x1.40mm_HandSolder, symbol Device:R
- Q1, Q2, Q3, Q4: Farnell (none) -> 3121715
- Q5, Q6: footprint Package_TO_SOT_THT:TO-220-3_Vertical -> esp-switch:TO-220-3_Vertical_offset
- R11, R26: value 200 -> 220
- U1, U6: Farnell (none) -> 3778033
Connections:
- net +3V3: now also J1.7 (Pin_7)
- net GND: now also J1.6 (Pin_6)
- net GPIO0: now also Q8.1 (C)
- net GPIO1: now also R31.2
- net GPIO10: now also R11.1; no longer C10.1, R15.2, U3.4
- net GPIO12: now also C11.1, R16.2, U4.4; no longer R11.1
- net GPIO13: now also C10.1, R15.2, U3.4; no longer R26.1
- net GPIO3: now also R34.1
- net GPIO9: now also R26.1; no longer C11.1, R16.2, U4.4
- net nRST: now also Q7.1 (C)
- net at J7.1 (Pin_1), R18.1: now also D4.2 (A2)
- net at J7.2 (Pin_2), R19.1: now also D4.1 (A1)
- net at J7.4 (Pin_4), R20.1: now also D5.2 (A2)
- net at J7.3 (Pin_3), R21.1: now also D5.1 (A1)
- net at R27.1, U6.4 (R): now also Q6.3 (G)
- net at R27.2: now also J2.4 (Pin_4), Q6.1 (A1), D7.2 (A2); no longer Q6.3 (G)
- net at J2.1 (Pin_1), Q5.1 (A1): now also R12.2, D6.2 (A2)
- net at J2.2 (Pin_2), Q5.2 (A2), R25.1: now also D6.1 (A1)
- net at Q5.3 (G): now also R12.1, U1.4 (R); no longer R12.2
- net at J2.3 (Pin_3), Q6.2 (A2), R28.1: now also D7.1 (A1)
- new net: Q8.3 (E), R29.1, R32.2
- new net: Q7.2 (B), R29.2
- new net: J1.1 (Pin_1), R33.1
- new net: J1.2 (Pin_2), R32.1
- new net: J1.3 (Pin_3), R31.1
- new net: J1.4 (Pin_4), R34.2
- new net: Q8.2 (B), R30.2
- new net: Q7.3 (E), R30.1, R33.2
- no-connect marks 6 -> 7
Other:
- moved on the sheet: C10, C11, C5, D1, D2, J7, Q5, Q6, R11, R12, R15, R16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

Commit message: Update values
Parts:
- R1: value 68k -> 150k
- R10, R13, R14, R2, R29, R3, R30, R4, R5, R6, R9: value 10k -> 22k
- R32, R33: value 220 -> 10R
Other:
- note added: "Check layout"
- note added: "TO GPIO16 and reverse polarity"
Changed lines of the file:
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@@
     (stroke (width 0) (type default))
+  )
+  (text "TO GPIO16 and reverse polarity" (at 116.84 144.145 0)
+    (effects (font (size 1.27 1.27)) (justify left bottom))
+  )
+  (text "Check layout" (at 202.565 27.305 0)
+    (effects (font (size 1.27 1.27)) (justify left bottom))
+  )
+  (text "Check layout" (at 199.39 58.42 0)
+    (effects (font (size 1.27 1.27)) (justify left bottom))
+  )
+  (text "Check layout" (at 78.74 87.63 0)
+    (effects (font (size 1.27 1.27)) (justify left bottom))
   )
   (label "GPIO3" (at 170.18 46.99 180) (fields_autoplaced)
@@
       (effects (font (size 1.27 1.27)))
     )
-    (property "Value" "10k" (at 40.64 183.7436 90)
+    (property "Value" "22k" (at 40.64 183.7436 90)
       (effects (font (size 1.27 1.27)))
     )
@@
       (effects (font (size 1.27 1.27)))
     )
-    (property "Value" "10k" (at 40.64 162.1536 90)
+    (property "Value" "22k" (at 40.64 162.1536 90)
       (effects (font (size 1.27 1.27)))
     )
@@
       (effects (font (size 1.27 1.27)))
     )
-    (property "Value" "10k" (at 40.64 140.5636 90)
+    (property "Value" "22k" (at 40.64 140.5636 90)
       (effects (font (size 1.27 1.27)))
     )
@@
       (effects (font (size 1.27 1.27)))
     )
-    (property "Value" "10k" (at 40.64 118.9736 90)
+    (property "Value" "22k" (at 40.64 118.9736 90)
       (effects (font (size 1.27 1.27)))
     )
@@
       (effects (font (size 1.27 1.27)) (justify right))
     )
-    (property "Value" "10k" (at 177.038 34.163 0)
+    (property "Value" "22k" (at 177.038 34.163 0)
       (effects (font (size 1.27 1.27)) (justify right))
     )
@@
       (effects (font (size 1.27 1.27)) (justify right))
     )
-    (property "Value" "10k" (at 184.658 34.163 0)
+    (property "Value" "22k" (at 184.658 34.163 0)
       (effects (font (size 1.27 1.27)) (justify right))
     )
@@
       (effects (font (size 1.27 1.27)) (justify right))
     )
-    (property "Value" "10k" (at 114.808 34.163 0)
+    (property "Value" "22k" (at 114.808 34.163 0)
       (effects (font (size 1.27 1.27)) (justify right))
     )
@@
       (effects (font (size 1.27 1.27)) (justify right))
     )
-    (property "Value" "10k" (at 126.238 34.163 0)
+    (property "Value" "22k" (at 126.238 34.163 0)
       (effects (font (size 1.27 1.27)) (justify right))
     )
@@
       (effects (font (size 1.27 1.27)) (justify left))
     )
-    (property "Value" "10k" (at 48.768 86.233 0)
+    (property "Value" "22k" (at 48.768 86.233 0)
       (effects (font (size 1.27 1.27)) (justify left))
     )
@@
       (effects (font (size 1.27 1.27)) (justify left))
     )
-    (property "Value" "68k" (at 48.768 73.533 0)
+    (property "Value" "150k" (at 48.768 73.533 0)
       (effects (font (size 1.27 1.27)) (justify left))
     )
@@
       (effects (font (size 1.27 1.27)))
     )
-    (property "Value" "10k" (at 238.76 122.7836 90)
+    (property "Value" "22k" (at 238.76 122.7836 90)
       (effects (font (size 1.27 1.27)))
     )
@@
       (effects (font (size 1.27 1.27)))
     )
-    (property "Value" "220" (at 252.095 128.6764 90)
+    (property "Value" "10R" (at 252.095 128.6764 90)
       (effects (font (size 1.27 1.27)))
     )
@@
       (effects (font (size 1.27 1.27)))
     )
-    (property "Value" "220" (at 252.095 147.0914 90)
+    (property "Value" "10R" (at 252.095 147.0914 90)
       (effects (font (size 1.27 1.27)))
     )
@@
       (effects (font (size 1.27 1.27)))
     )
-    (property "Value" "10k" (at 238.76 141.1986 90)
-      (effects (font (size 1.27 1.27)))
-    )
+    (property "Value" "22k" (at 238.76 141.1986 90)
+      (effects (font (size 1.27 1.27)))
+    )

Commit message: Updates
Parts:
- Q5, Q6: footprint esp-switch:TO-220-3_Vertical_offset -> Package_TO_SOT_SMD:TO-252-2
Connections:
- net GND: now also R11.1, R26.1; no longer U1.2 (K), U6.2 (K)
- net GPIO0: now also Q2.1 (G), R4.2
- net GPIO10: no longer R11.1
- net GPIO2: now also Q1.1 (G), R3.2
- net GPIO4: now also U6.1 (A); no longer Q2.1 (G), R4.2
- net GPIO5: now also U1.1 (A); no longer Q1.1 (G), R3.2
- net GPIO9: no longer R26.1
- net at Q6.1 (A1), R27.2: now also D7.1 (A1), J2.3 (Pin_3); no longer D7.2 (A2), J2.4 (Pin_4)
- net at Q5.1 (A1), R12.2: now also D6.1 (A1), J2.2 (Pin_2); no longer D6.2 (A2), J2.1 (Pin_1)
- net at Q5.2 (A2), R25.1: now also D6.2 (A2), J2.1 (Pin_1); no longer D6.1 (A1), J2.2 (Pin_2)
- net at Q6.2 (A2), R28.1: now also D7.2 (A2), J2.4 (Pin_4); no longer D7.1 (A1), J2.3 (Pin_3)
- net at R26.2: now also U6.2 (K); no longer U6.1 (A)
- net at R11.2: now also U1.2 (K); no longer U1.1 (A)
Other:
- note added: "Incorrect footprint"
- note removed: "TO GPIO16 and reverse polarity"
- moved on the sheet: D6, D7, R11, R26
